File: Reversible Keyboard.kicad_sch (KiCad schematic)
At the start: 106 parts, among them SW1 Push_Button, SW2 Push_Button, SW3 SW_SPDT, SW4 SW_SPDT, U2 Seeed Studio XIAO SAMD21

Commit message: Uploaded Libraries
Parts:
- BT1: symbol Device:Battery_Cell -> Library:Battery_Cell
- D1, D10, D11, D12, D13, D14, D15, D16, D17, D18, D19, D2, D20, D21, D22, D23, D24, D25, D26, D27, D28, D29, D3, D30, D31, D32, D33, D34, D35, D36, D37, D38, D39, D4, D40, D41, D42, D43, D44, D45, D46, D47, D48, D49, D5, D50, D51, D52, D53, D54, D55, D56, D57, D58, D59, D6, D60, D7, D8, D9: symbol Device:D -> Library:D
- H1, H2, H3, H4, H5, H6, H7, H8, H9: symbol Mechanical:MountingHole -> Library:MountingHole
- S1, S10, S11, S12, S13, S14, S15, S16, S17, S18, S19, S2, S20, S21, S22, S23, S24, S25, S26, S27, S28, S29, S3, S30, S4, S5, S6, S7, S8, S9: symbol s-ol:PG1350 -> Library:PG1350
- SW1, SW2: symbol PCM_SL_Devices:Push_Button -> Library:Push_Button
- SW3, SW4: symbol Switch:SW_SPDT -> Library:SW_SPDT
